File: relays.kicad_sch (KiCad schematic)
At the start: 0 parts

Commit message: Finished schematics, started component placement
Parts:
- added C1, C2: 10u, Capacitor_SMD:C_0603_1608Metric, symbol Device:C
- added D6, D7, D8: ~, EasyEDA_Lib:SOD-123_L2.7-W1.6-LS3.7-RD, symbol EasyEDA_Lib:1N5819HW-7-F
- added H6, H7, H8: ~, EasyEDA_Lib:HDR-TH_2P-P2.54-V-F, symbol EasyEDA_Lib:ZX-PM2.54-1-2PY
- added Q2, Q3, Q4: ~, EasyEDA_Lib:SOT-23-3_L2.9-W1.6-P1.90-LS2.8-BR, symbol EasyEDA_Lib:BC817-40,215
- added R10, R13, R16: 1K, Resistor_SMD:R_0603_1608Metric, symbol Device:R
- added R11, R14, R17: 10K, Resistor_SMD:R_0603_1608Metric, symbol Device:R
- added R12, R15, R18: 10R, Resistor_THT:R_Axial_DIN0516_L15.5mm_D5.0mm_P20.32mm_Horizontal, symbol Device:R
- added RLY1, RLY2, RLY3: ~, EasyEDA_Lib:RELAY-TH_G5NB-1A-E-DCXX, symbol EasyEDA_Lib:G5NB-1A-E-DC12
- added U2: ~, EasyEDA_Lib:SOT-223_L6.3-W3.5-P2.30-LS7.0-BR, symbol EasyEDA_Lib:SSP7903P12FR
Connections:
- new net: H6.1, RLY1.2
- new net: Q2.1, R10.2, R11.1
- new net: D8.2 (A), Q4.3, RLY3.1
- new net: H7.1, RLY2.2
- new net: Q4.1, R16.2, R17.1
- new net: Q3.1, R13.2, R14.1
- new net: H8.1, RLY3.2
- new net: R18.2, RLY3.3
- new net: D6.2 (A), Q2.3, RLY1.1
- new net: R12.2, RLY1.3
- new net: R15.2, RLY2.3
- new net: D7.2 (A), Q3.3, RLY2.1
- new net GND: C1.2, C2.2, H6.2, H7.2, H8.2, Q2.2, Q3.2, Q4.2, R11.2, R14.2, R17.2, U2.1 (GND)
- new net RELAY1: R10.1
- new net RELAY2: R13.1
- new net RELAY3: R16.1
- new net VCC: C2.1, R12.1, R15.1, R18.1, U2.3 (VIN)
- new net Vdrive: C1.1, D6.1 (K), D7.1 (K), D8.1 (K), RLY1.4, RLY2.4, RLY3.4, U2.2 (VOUT), U2.4 (VOUT)

Commit message: Pretty much finished the PCB, only got the silkscreen decorations left
Parts:
- added D10, D11, D12: LED, LED_SMD:LED_0603_1608Metric, symbol Device:LED
- added R30, R31, R32: 1K, Resistor_SMD:R_0603_1608Metric, symbol Device:R
Connections:
- net GND: now also D10.1 (K), D11.1 (K), D12.1 (K)
- net RELAY1: now also R30.2
- net RELAY2: now also R31.2
- net RELAY3: now also R32.2
- new net: D10.2 (A), R30.1
- new net: D11.2 (A), R31.1
- new net: D12.2 (A), R32.1
