File: pcb/power.kicad_sch (KiCad schematic)
At the start: 3 parts

Commit message: Upgrade kicad version to 10, add krita capacitor image
Parts:
- D3, DC1, H2: value ~ -> (none)

Commit message: Add JLC carts and BOM
Parts:
- D3: Supplier Part URL (none) -> https://www.lcsc.com/product-detail/C85098.html
- DC1: Supplier Part URL (none) -> https://www.lcsc.com/product-detail/C720557.html
- H2: now left out of the parts list
Changed lines of the file:
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@@
 		(body_style 1)
 		(exclude_from_sim no)
-		(in_bom yes)
+		(in_bom no)
 		(on_board yes)
 		(in_pos_files yes)
@@
 		)
 		(property "LCSC Part Name" "1x2P 间距:2.54mm 方针 直插"
+			(at 127 97.79 0)
+			(hide yes)
+			(show_name no)
+			(do_not_autoplace no)
+			(effects
+				(font
+					(size 1.27 1.27)
+				)
+			)
+		)
+		(property "Supplier Part URL" ""
 			(at 127 97.79 0)
 			(hide yes)
@@
 			)
 		)
+		(property "Supplier Part URL" "https://www.lcsc.com/product-detail/C720557.html"
+			(at 48.26 46.99 0)
+			(hide yes)
+			(show_name no)
+			(do_not_autoplace no)
+			(effects
+				(font
+					(size 1.27 1.27)
+				)
+			)
+		)
 		(pin "2"
 		)
@@
 			(at 125.73 52.07 0)
 			(hide yes)
+			(show_name no)
+			(do_not_autoplace no)
+			(effects
+				(font
+					(size 1.27 1.27)
+				)
+			)
+		)
+		(property "Supplier Part URL" "https://www.lcsc.com/product-detail/C85098.html"
+			(at 125.73 52.07 0)
+			(hide yes)
